File: _saved_power.sch (KiCad schematic (older format))
At the start: 0 parts

Commit message: hiearchic
Parts:
- added C13, C19: 1n, Capacitor_SMD:C_0805_2012Metric, symbol Device:C
- added C14: 100p, Capacitor_SMD:C_0805_2012Metric, symbol Device:C
- added C20, C24, C25, C27, C7: 100n, Capacitor_SMD:C_0805_2012Metric, symbol Device:C
- added C21: 100u, Capacitor_THT:CP_Radial_D10.0mm_P5.00mm, symbol Device:CP
- added C22: 4u7, Capacitor_SMD:C_0805_2012Metric, symbol Device:C
- added C23: 1u, Capacitor_SMD:C_0805_2012Metric, symbol Device:C
- added C26: 470u, Capacitor_THT:CP_Radial_D10.0mm_P5.00mm, symbol Device:CP
- added C28, C38, C39: NFM21CC223R1H3D, EMI_Suppression_Filters_Cap_Type:NFM21C_Series, symbol Device:EMI_Filter_C
- added C3: 47u, Capacitor_THT:CP_Radial_D5.0mm_P2.50mm, symbol Device:CP
- added C9: 10n, Capacitor_SMD:C_0805_2012Metric, symbol Device:C
- added D6: STPS3L60U, Diode_SMD:D_SMB, symbol Device:D_Schottky
- added D_50V1, D_5V1: LH R974-LP-1, LED_SMD:LED_0805_2012Metric, symbol Device:LED
- added J10: 50V_OUT, KLALIB_PCB_Screw_Terminal:TerminalBlock_KEYS7808, symbol Connector_Generic:Conn_01x01
- added J12, J14, J15, J16, J18, J19: 50V_GND, MountingHole:MountingHole_3.2mm_M3_Pad_Via, symbol Connector_Generic:Conn_01x01
- added J9: 50V_IN, KLALIB_PCB_Screw_Terminal:TerminalBlock_KEYS7808, symbol Connector_Generic:Conn_01x01
- added L4: DE1209-230u, Inductor_SMD:L_12x12mm_H8mm, symbol Device:L
- added L5, L7, L8: BLM31PG500SN1L, Capacitor_SMD:C_1206_3216Metric, symbol Device:Ferrite_Bead
- added Q2: BSS138, Package_TO_SOT_SMD:SOT-23, symbol Device:Q_NMOS_GSD
- added Q5: BBS3002-TL-1E, Package_TO_SOT_SMD:TO-263-2, symbol Device:Q_PMOS_GDS
- added R13: 499R, Resistor_SMD:R_0805_2012Metric, symbol Device:R
- added R14, R16: 10k, Resistor_SMD:R_0805_2012Metric, symbol Device:R
- added R15: 270k, Resistor_SMD:R_0805_2012Metric, symbol Device:R
- added R18: 100k, Resistor_SMD:R_0805_2012Metric, symbol Device:R
- added R19, R20: 0R005, KLALIB_Resistors_Shunt:OAR5R010FLF, symbol Device:R
- added R22: 4k7, Resistor_SMD:R_0805_2012Metric, symbol Device:R
- added R27: 12k, Resistor_SMD:R_0805_2012Metric, symbol Device:R
- added R28: 18k, Resistor_SMD:R_0805_2012Metric, symbol Device:R
- added R9: 1k, Resistor_SMD:R_0805_2012Metric, symbol Device:R
- added TP1: ADC_UCC, TestPoint:TestPoint_Pad_D2.0mm, symbol Connector_Generic:Conn_01x01
- added TP2: +5V, TestPoint:TestPoint_Pad_D2.0mm, symbol Connector_Generic:Conn_01x01
- added TP3: +12V, TestPoint:TestPoint_Pad_D2.0mm, symbol Connector_Generic:Conn_01x01
- added TP4: ADC ICC, TestPoint:TestPoint_Pad_D2.0mm, symbol Connector_Generic:Conn_01x01
- added TP5: GND, TestPoint:TestPoint_Pad_D2.0mm, symbol Connector_Generic:Conn_01x01
- added U2: LP2950-5.0_TO252, Package_TO_SOT_SMD:TO-252-2, symbol Regulator_Linear:LP2950-5.0_TO252
- added U3: LM2576HVS-12, Package_TO_SOT_SMD:TO-263-5_TabPin3, symbol Regulator_Switching:LM2576HVS-12
- added U4: LTC6101AHS5, Package_TO_SOT_SMD:SOT-23-5, symbol KLALIB_Amplifiers:LTC6101AHS5
Connections:
- net labels added: +12V, +50V, +5V, ADC_ICC, ADC_UCC, GND, MCU_SUPPLY
- wire segments 0 -> 78
Other:
- note added: "0,1V @ 40A\nPztr 4W"
- note added: "For gain 20\nR13 = 499R\nR14 = 10k"
