File: _saved_sekvencer_v0.01.sch (KiCad schematic (older format))
At the start: 139 parts, among them J1 AVR_ISP_01X06, J10 50V_OUT, J11 BIAS_DIRECT, J12 50V_GND, J13 TERMISTOR, J14 50V_GND, J15 50V_GND, J16 50V_GND, J17 BIAS, J18 50V_GND, J19 50V_GND, J2 PTT, J3 SWR, J4 POWER, J5 LCD, J6 RX_REL, J7 TX_REL, J8 FAN, J9 50V_IN, Q1 BC857, Q2 BSS138, Q3 BSS138, Q4 IRLML0030TRPBF, Q5 BBS3002-TL-1E, Q6 BSS138, Q7 BC847, U1 ATmega328P-AU, U2 LP2950-5.0_TO252, U3 LM2576HVS-12, U4 LTC6101AHS5, U5 LP2951ACD-3.3R2G, Y1 LFXTAL071268CUTT 16MHz

Commit message: hiearchic
Parts:
- removed C13, C19: 1n, Capacitor_SMD:C_0805_2012Metric, symbol Device:C
- removed C14: 100p, Capacitor_SMD:C_0805_2012Metric, symbol Device:C
- removed C20, C24, C25, C27, C7: 100n, Capacitor_SMD:C_0805_2012Metric, symbol Device:C
- removed C21: 100u, Capacitor_THT:CP_Radial_D10.0mm_P5.00mm, symbol Device:CP
- removed C22: 4u7, Capacitor_SMD:C_0805_2012Metric, symbol Device:C
- removed C23: 1u, Capacitor_SMD:C_0805_2012Metric, symbol Device:C
- removed C26: 470u, Capacitor_THT:CP_Radial_D10.0mm_P5.00mm, symbol Device:CP
- removed C28, C38, C39: NFM21CC223R1H3D, EMI_Suppression_Filters_Cap_Type:NFM21C_Series, symbol Device:EMI_Filter_C
- removed C3: 47u, Capacitor_THT:CP_Radial_D5.0mm_P2.50mm, symbol Device:CP
- removed C9: 10n, Capacitor_SMD:C_0805_2012Metric, symbol Device:C
- removed D6: STPS3L60U, Diode_SMD:D_SMB, symbol Device:D_Schottky
- removed D_50V1, D_5V1: LH R974-LP-1, LED_SMD:LED_0805_2012Metric, symbol Device:LED
- removed J10: 50V_OUT, KLALIB_PCB_Screw_Terminal:TerminalBlock_KEYS7808, symbol Connector_Generic:Conn_01x01
- removed J12, J14, J15, J16, J18, J19: 50V_GND, MountingHole:MountingHole_3.2mm_M3_Pad_Via, symbol Connector_Generic:Conn_01x01
- removed J9: 50V_IN, KLALIB_PCB_Screw_Terminal:TerminalBlock_KEYS7808, symbol Connector_Generic:Conn_01x01
- removed L4: DE1209-230u, Inductor_SMD:L_12x12mm_H8mm, symbol Device:L
- removed L5, L7, L8: BLM31PG500SN1L, Capacitor_SMD:C_1206_3216Metric, symbol Device:Ferrite_Bead
- removed Q2: BSS138, Package_TO_SOT_SMD:SOT-23, symbol Device:Q_NMOS_GSD
- removed Q5: BBS3002-TL-1E, Package_TO_SOT_SMD:TO-263-2, symbol Device:Q_PMOS_GDS
- removed R13: 499R, Resistor_SMD:R_0805_2012Metric, symbol Device:R
- removed R14, R16: 10k, Resistor_SMD:R_0805_2012Metric, symbol Device:R
- removed R15: 270k, Resistor_SMD:R_0805_2012Metric, symbol Device:R
- removed R18: 100k, Resistor_SMD:R_0805_2012Metric, symbol Device:R
- removed R19, R20: 0R005, KLALIB_Resistors_Shunt:OAR5R010FLF, symbol Device:R
- removed R22: 4k7, Resistor_SMD:R_0805_2012Metric, symbol Device:R
- removed R27: 12k, Resistor_SMD:R_0805_2012Metric, symbol Device:R
- removed R28: 18k, Resistor_SMD:R_0805_2012Metric, symbol Device:R
- removed R9: 1k, Resistor_SMD:R_0805_2012Metric, symbol Device:R
- removed TP1: ADC_UCC, TestPoint:TestPoint_Pad_D2.0mm, symbol Connector_Generic:Conn_01x01
- removed TP2: +5V, TestPoint:TestPoint_Pad_D2.0mm, symbol Connector_Generic:Conn_01x01
- removed TP3: +12V, TestPoint:TestPoint_Pad_D2.0mm, symbol Connector_Generic:Conn_01x01
- removed TP4: ADC ICC, TestPoint:TestPoint_Pad_D2.0mm, symbol Connector_Generic:Conn_01x01
- removed TP5: GND, TestPoint:TestPoint_Pad_D2.0mm, symbol Connector_Generic:Conn_01x01
- removed U2: LP2950-5.0_TO252, Package_TO_SOT_SMD:TO-252-2, symbol Regulator_Linear:LP2950-5.0_TO252
- removed U3: LM2576HVS-12, Package_TO_SOT_SMD:TO-263-5_TabPin3, symbol Regulator_Switching:LM2576HVS-12
- removed U4: LTC6101AHS5, Package_TO_SOT_SMD:SOT-23-5, symbol KLALIB_Amplifiers:LTC6101AHS5
Connections:
- net labels removed: +50V
- wire segments 222 -> 149
Other:
- note removed: "0,1V @ 40A\nPztr 4W"
- note removed: "For gain 20\nR13 = 499R\nR14 = 10k"
