File: power.sch (KiCad schematic (older format))
At the start: 14 parts

Commit message: hiearchic
Parts:
- removed C?: 10n, Capacitor_SMD:C_0805_2012Metric, symbol Device:C
- removed C?: 1n, Capacitor_SMD:C_0805_2012Metric, symbol Device:C
- removed C?: 100p, Capacitor_SMD:C_0805_2012Metric, symbol Device:C
- removed C?: 100u, Capacitor_THT:CP_Radial_D10.0mm_P5.00mm, symbol Device:CP
- removed C? (x2): 100n, Capacitor_SMD:C_0805_2012Metric, symbol Device:C
- removed C?: 470u, Capacitor_THT:CP_Radial_D10.0mm_P5.00mm, symbol Device:CP
- removed C?: NFM21CC223R1H3D, EMI_Suppression_Filters_Cap_Type:NFM21C_Series, symbol Device:EMI_Filter_C
- removed D?: STPS3L60U, Diode_SMD:D_SMB, symbol Device:D_Schottky
- removed L?: DE1209-230u, Inductor_SMD:L_12x12mm_H8mm, symbol Device:L
- removed L?: BLM31PG500SN1L, Capacitor_SMD:C_1206_3216Metric, symbol Device:Ferrite_Bead
- removed R?: 270k, Resistor_SMD:R_0805_2012Metric, symbol Device:R
- removed R?: 10k, Resistor_SMD:R_0805_2012Metric, symbol Device:R
- removed U?: LM2576HVS-12, Package_TO_SOT_SMD:TO-263-5_TabPin3, symbol Regulator_Switching:LM2576HVS-12
- added C13: 1n, Capacitor_SMD:C_0805_2012Metric, symbol Device:C
- added C14: 100p, Capacitor_SMD:C_0805_2012Metric, symbol Device:C
- added C20, C27: 100n, Capacitor_SMD:C_0805_2012Metric, symbol Device:C
- added C21: 100u, Capacitor_THT:CP_Radial_D10.0mm_P5.00mm, symbol Device:CP
- added C26: 470u, Capacitor_THT:CP_Radial_D10.0mm_P5.00mm, symbol Device:CP
- added C28: NFM21CC223R1H3D, EMI_Suppression_Filters_Cap_Type:NFM21C_Series, symbol Device:EMI_Filter_C
- added C9: 10n, Capacitor_SMD:C_0805_2012Metric, symbol Device:C
- added D6: STPS3L60U, Diode_SMD:D_SMB, symbol Device:D_Schottky
- added L4: DE1209-230u, Inductor_SMD:L_12x12mm_H8mm, symbol Device:L
- added L5: BLM31PG500SN1L, Capacitor_SMD:C_1206_3216Metric, symbol Device:Ferrite_Bead
- added R15: 270k, Resistor_SMD:R_0805_2012Metric, symbol Device:R
- added R16: 10k, Resistor_SMD:R_0805_2012Metric, symbol Device:R
- added TP1: ADC_UCC, TestPoint:TestPoint_Pad_D2.0mm, symbol Connector_Generic:Conn_01x01
- added TP3: +12V, TestPoint:TestPoint_Pad_D2.0mm, symbol Connector_Generic:Conn_01x01
- added U3: LM2576HVS-12, Package_TO_SOT_SMD:TO-263-5_TabPin3, symbol Regulator_Switching:LM2576HVS-12
Connections:
- wire segments 26 -> 27
